Commit message: feat: add sensor livox mid-360

File: urdf/raspicat.urdf.xacro (robot description, xacro)
@@ -6,16 +6,16 @@
   <!-- =============== Xacro arg =============== -->
   <xacro:arg name="gazebo_plugin"         default="true"/>
-  <xacro:arg name="camera_gazebo_plugin"  default="true"/>
+  <xacro:arg name="camera_gazebo_plugin"  default="false"/>
   <xacro:arg name="imu_gazebo_plugin"     default="true"/>
   <xacro:arg name="diffdrive_pub_tf"      default="true"/>
   <xacro:arg name="jointstate"            default="true"/>
   <xacro:arg name="laser_visual"          default="false"/>
-  <xacro:arg name="ultrasonic_visual"     default="true"/>
+  <xacro:arg name="ultrasonic_visual"     default="false"/>
   <xacro:arg name="robot_namespace"       default=""/>
   <xacro:arg name="diffdrive_namespace"   default="/"/>
-  <xacro:arg name="lidar_frame"           default="lidar_link"/>
+  <xacro:arg name="lidar_frame"           default="livox_frame"/>
   <!-- =============== Xacro property =============== -->
-  <xacro:property name="lidar_mount_z" value="0.0"/>
-  <xacro:property name="lidar_sensor_z" value="0.055"/>
+  <xacro:property name="lidar_mount_z" value="0.7"/>
+  <xacro:property name="lidar_sensor_z" value="0.047"/>
   <!-- =============== Xacro include =============== -->
   <xacro:include filename="$(find raspicat_description)/urdf/common.xacro"/>
@@ -53,5 +53,5 @@
   <!-- Sensors -->
   <xacro:lidar_mount prefix="lidar_mount" parent="base_link">
-    <origin xyz="0.144 0 ${lidar_mount_z - 0.0262}" rpy="0 0 0"/>
+    <origin xyz="-0.365 0 ${lidar_mount_z - 0.0262}" rpy="${M_PI} 0 0"/>
   </xacro:lidar_mount>
   <xacro:lidar_sensor prefix="laser" parent="lidar_mount_link" lidar_frame="$(arg lidar_frame)">
@@ -92,5 +92,5 @@
     <!-- Sensors -->
     <xacro:lidar_gazebo lidar_frame="$(arg lidar_frame)"
-      min_angle="-1.9" max_angle="1.9" min_range="0.1" max_range="30" visualize="$(arg laser_visual)"/>
+      min_angle="-1.9" max_angle="1.9" min_range="0.1" max_range="80" visualize="$(arg laser_visual)"/>
     <xacro:ultrasonic_sensor_gazebo prefix="right_side"
       min_angle="-0.0574533" max_angle="0.0574533" min_range="0.02" max_range="4.095" visualize="$(arg ultrasonic_visual)"/>

File: urdf/sensors/lidar.gazebo.xacro (robot description, xacro)
@@ -6,13 +6,19 @@
         <pose>0 0 0 0 0 0</pose>
         <visualize>${visualize}</visualize>
-        <update_rate>30</update_rate>
+        <update_rate>10</update_rate>
         <ray>
           <scan>
             <horizontal>
-              <samples>720</samples>
+              <samples>100</samples>
               <resolution>1</resolution>
-              <min_angle>${min_angle}</min_angle>
-              <max_angle>${max_angle}</max_angle>
+              <min_angle>${M_PI}</min_angle>
+              <max_angle>-${M_PI}</max_angle>
             </horizontal>
+            <vertical>
+              <samples>50</samples>
+              <resolution>1</resolution>
+              <min_angle>-0.1221730476396</min_angle>
+              <max_angle>0.90757121103706</max_angle>
+            </vertical>
           </scan>
           <range>
@@ -29,8 +35,8 @@
         <plugin name="gazebo_ros_${lidar_frame}_controller" filename="libgazebo_ros_ray_sensor.so">
           <ros>
-            <remapping>~/out:=scan</remapping>
+            <remapping>~/out:=/livox/lidar</remapping>
           </ros>
           <frame_name>lidar_link</frame_name>
-          <output_type>sensor_msgs/LaserScan</output_type>
+          <output_type>sensor_msgs/PointCloud2</output_type>
         </plugin>
       </sensor>

File: urdf/sensors/lidar.urdf.xacro (robot description, xacro)
@@ -2,4 +2,7 @@
 <robot name="raspicat_lidar_sensor" xmlns:xacro="http://ros.org/wiki/xacro">
   <xacro:include filename="$(find raspicat_description)/urdf/sensors/lidar.gazebo.xacro"/>
+  <material name="gray">
+    <color rgba="0.5 0.5 0.5 1.0"/>
+  </material>
   <xacro:macro name="lidar_mount" params="prefix parent *joint_origin">
     <joint name="${prefix}_joint" type="fixed">
@@ -16,5 +19,13 @@
       <child link="${lidar_frame}"/>
     </joint>
-    <link name="${lidar_frame}"/>
+    <link name="${lidar_frame}">
+      <visual>
+        <origin xyz="0 0 0" rpy="${M_PI/2} 0 0"/>
+        <geometry>
+          <mesh filename="package://raspicat_description/meshes/stl/sensors/mid-360.stl" scale="0.001 0.001 0.001"/>
+        </geometry>
+        <material name="gray"/>
+      </visual>
+    </link>
   </xacro:macro>
 </robot>
